Commit message: delete old box, add new; compile and generate joint limits, exclude contacts.

File: assets/mj_plain_sw/plain_sw.urdf (robot description, URDF)
Before this commit: robot Plain_Box_URDF, 2 links, 1 joints
Links:
- link base_link: mass 0.65846 -> 0.658458282652952; geometry collision mesh filename=package://plain_sw/meshes/base_link.STL; visual mesh filename=package://plain_sw/meshes/base_link.STL
- link top_Link: mass 0.40215 -> 0.40215431638902; geometry collision mesh filename=package://plain_sw/meshes/top_Link.STL; visual mesh filename=package://plain_sw/meshes/top_Link.STL
Joints:
- joint joint_1: axis 0 0 1 -> 0 0 -1; limit lower=0 upper=2 effort=100 velocity=10 -> lower=-2 upper=2 effort=100 velocity=10; origin xyz=0 -0.0050165 0.071196 rpy=2.8878 0 0 -> xyz=0 0.071183 0.14422 rpy=1.5708 0 -1.5708

File: assets/plain_sw/urdf/plain_sw.urdf (robot description, URDF)
Before this commit: robot Plain_Box_URDF, 2 links, 1 joints
Links:
- link base_link: mass 0.65846 -> 0.658458282652952; geometry collision mesh filename=package://plain_sw/meshes/base_link.STL; visual mesh filename=package://plain_sw/meshes/base_link.STL
- link top_Link: mass 0.40215 -> 0.40215431638902; geometry collision mesh filename=package://plain_sw/meshes/top_Link.STL; visual mesh filename=package://plain_sw/meshes/top_Link.STL
Joints:
- joint joint_1: axis 0 0 1 -> 0 0 -1; limit lower=0 upper=2 effort=100 velocity=10 -> lower=-2 upper=2 effort=100 velocity=10; origin xyz=0 -0.0050165 0.071196 rpy=1.57079632679 0 0 -> xyz=0 0.071183 0.14422 rpy=1.5708 0 -1.5708
